File: solar-cells/solar-cell-pcbs-usb/solar-cell-pcbs-usb.kicad_pcb (KiCad board)
At the start: 2 copper layers, 80 x 103.5 mm, 18 parts, among them J1 Solar Cell, J2 Burn Wire

Commit message: modifications to solar cell folder
Parts:
- removed J2: Burn Wire, Molex_PicoLock_2p_2mm_2053380002:2053380002
- removed LowerBurn1, UpperBurn1: Burn+, TestPoint:TestPoint_Pad_2.0x2.0mm
- removed LowerBurn2, UpperBurn2: Burn-, TestPoint:TestPoint_Pad_2.0x2.0mm
- SC1, SC2: footprint TestPoint:TestPoint_Pad_D3.0mm -> TestPoint:TestPoint_THTPad_D3.0mm_Drill1.5mm
- moved J1 41.7 mm to (86.3, 111.4)
- moved SC1 10.8 mm to (90.0, 71.8)
- moved SC2 10.8 mm to (134.3, 71.8)
- moved TP1 6.10 mm to (71.8, 53.2)
- moved TP2 6.10 mm to (71.7, 48.3)
Routing:
- net SC-: track 0.00 -> 163.9 mm
- net SC+: track 9.21 -> 76.8 mm, vias 1 -> 0
- net BURN+: track 36.4 -> 0.00 mm, vias 2 -> 0
- net BURN-: track 34.4 -> 0.00 mm, vias 2 -> 0
Other:
- board size 80 x 103.5 mm -> 89 x 103.5 mm
- board text added: "RBF Pin"
- board text added: "Solar Cell"
- board text added: "USB-C"
