File: solar-cells/solar cell non-usb side/solar-cell-pcbs-usb.kicad_pcb (KiCad board)
At the start: 2 copper layers, 80 x 103.5 mm, 13 parts, among them J1 Solar Cell

Commit message: modify non usb pcb
Connections:
- net SC- renamed GND
Routing:
- net GND: track 76.9 -> 0.00 mm
- added copper zone on B.Cu, net GND
Other:
- board text added: "Solar Cell"
Changed lines of the file:
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@@
   )
   (net 0 "")
-  (net 1 "SC-")
+  (net 1 "GND")
   (net 2 "SC+")
   (footprint "TestPoint:TestPoint_Loop_D1.80mm_Drill1.0mm_Beaded" (layer "F.Cu")
@@
       (effects (font (size 1 1) (thickness 0.15)))
     )
-    (fp_text value "SC+" (at 0 3.1) (layer "F.SilkS")
+    (fp_text value "SC+" (at 3.4 0 90) (layer "F.SilkS")
       (effects (font (size 1 1) (thickness 0.15)))
     )
@@
     (fp_circle (center 0 0) (end 1.3 0) (layer "F.Fab") (width 0.12) (fill none))
     (pad "1" thru_hole circle (at 0 -0.1) (size 2 2) (drill 1) (layers *.Cu *.Mask)
-      (net 1 "SC-") (pinfunction "1") (pintype "passive"))
+      (net 1 "GND") (pinfunction "1") (pintype "passive"))
     (model "${KICAD6_3DMODEL_DIR}/TestPoint.3dshapes/TestPoint_Loop_D1.80mm_Drill1.0mm_Beaded.wrl"
       (offset (xyz 0 0 0))
@@
       (effects (font (size 1 1) (thickness 0.15)))
     )
-    (fp_text value "SC-" (at 0 3.05) (layer "F.SilkS")
+    (fp_text value "SC-" (at 3.4 -0.025 90) (layer "F.SilkS")
       (effects (font (size 1 1) (thickness 0.15)))
     )
@@
     (fp_circle (center 0 0) (end 2 0) (layer "F.CrtYd") (width 0.05) (fill none))
     (pad "1" thru_hole circle (at 0 0) (size 3 3) (drill 1.5) (layers *.Cu *.Mask)
-      (net 1 "SC-") (pinfunction "1") (pintype "passive"))
+      (net 1 "GND") (pinfunction "1") (pintype "passive"))
   )
   (footprint "MountingHole:MountingHole_3.2mm_M3_DIN965_Pad" (layer "F.Cu")
@@
     (fp_line (start 5.152992 0.635) (end 5.152992 -0.635) (layer "B.Fab") (width 0.1))
     (pad "1" smd rect (at 0 0) (size 1.1 1.45) (layers "B.Cu" "B.Paste" "B.Mask")
-      (net 1 "SC-") (pinfunction "Pin_1") (pintype "passive"))
+      (net 1 "GND") (pinfunction "Pin_1") (pintype "passive"))
     (pad "2" smd rect (at -2.000001 0) (size 1.1 1.45) (layers "B.Cu" "B.Paste" "B.Mask")
       (net 2 "SC+") (pinfunction "Pin_2") (pintype "passive"))
@@
   (gr_line (start 80.65 38.75) (end 72.1 38.75) (layer "Edge.Cuts") (width 0.1))
   (gr_line (start 72.1 142.25) (end 72.1 38.75) (layer "Edge.Cuts") (width 0.1))
-  (gr_text "-" (at 97.5 113.25 -180) (layer "B.SilkS")
+  (gr_text "-" (at 97 113.65 -180) (layer "B.SilkS")
     (effects (font (size 1.5 1.5) (thickness 0.3)) (justify mirror))
   )
-  (gr_text "+" (at 94.5 113) (layer "B.SilkS")
+  (gr_text "+" (at 95.025 113.425) (layer "B.SilkS")
     (effects (font (size 1.5 1.5) (thickness 0.3)) (justify mirror))
+  )
+  (gr_text "Solar Cell" (at 112.95 132) (layer "F.SilkS")
+    (effects (font (size 1.5 1.5) (thickness 0.3)))
   )
   (dimension (type aligned) (layer "Dwgs.User")
@@
     (style (thickness 0.15) (arrow_length 1.27) (text_position_mode 0) (extension_height 0.58642) (extension_offset 0.5) keep_text_aligned)
   )
-  (segment (start 82.6 54.85) (end 76 48.25) (width 1.27) (layer "B.Cu") (net 1))
-  (segment (start 96.75 116.25) (end 97 116.5) (width 1.27) (layer "B.Cu") (net 1))
-  (segment (start 82.6 68.3) (end 82.6 54.85) (width 1.27) (layer "B.Cu") (net 1))
-  (segment (start 82.6 85.35) (end 96.75 99.5) (width 1.27) (layer "B.Cu") (net 1))
-  (segment (start 82.6 68.3) (end 82.6 85.35) (width 1.27) (layer "B.Cu") (net 1))
-  (segment (start 96.75 99.5) (end 96.75 116.25) (width 1.27) (layer "B.Cu") (net 1))
   (segment (start 91.199999 112.7) (end 82.6 112.7) (width 1.27) (layer "B.Cu") (net 2))
   (segment (start 94.999999 116.5) (end 91.199999 112.7) (width 1.27) (layer "B.Cu") (net 2))
   (segment (start 75.95 106.05) (end 75.95 53.25) (width 1.27) (layer "B.Cu") (net 2))
   (segment (start 82.6 112.7) (end 75.95 106.05) (width 1.27) (layer "B.Cu") (net 2))
+  (zone (net 1) (net_name "GND") (layer "B.Cu") (hatch edge 0.508)
+    (connect_pads (clearance 0.508))
+    (min_thickness 0.254) (filled_areas_thickness no)
+    (fill yes (thermal_gap 0.508) (thermal_bridge_width 0.508))
+    (polygon
+      (pts
+        (xy 152.9 37.775)
+        (xy 153.075 143.475)
+        (xy 70.975 143.5)
+        (xy 70.925 37.625)
+        (xy 70.925 37.6)
+      )
+    )
+  )
 )
