File: solar-cells/solar cell non-usb side/solar-cell-pcbs-usb.kicad_sch (KiCad schematic)
At the start: 13 parts, among them J1 Solar Cell

Commit message: modify non usb pcb
Connections:
- net SC- renamed GND
Changed lines of the file:
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@@
     (rev "1")
   )
+  (wire (pts (xy 45.72 58.42) (xy 44.45 58.42))
+    (stroke (width 0) (type default) (color 0 0 0 0))
+  )
   (wire (pts (xy 129.54 73.66) (xy 119.38 73.66))
     (stroke (width 0) (type default) (color 0 0 0 0))
   )
-  (wire (pts (xy 129.54 80.01) (xy 119.38 80.01))
+  (wire (pts (xy 120.65 62.23) (xy 121.92 62.23))
+    (stroke (width 0) (type default) (color 0 0 0 0))
+  )
+  (wire (pts (xy 119.38 80.01) (xy 121.92 80.01))
     (stroke (width 0) (type default) (color 0 0 0 0))
   )
   (wire (pts (xy 129.54 59.69) (xy 120.65 59.69))
-    (stroke (width 0) (type default) (color 0 0 0 0))
-  )
-  (wire (pts (xy 129.54 62.23) (xy 120.65 62.23))
     (stroke (width 0) (type default) (color 0 0 0 0))
   )
@@
     (effects (font (size 1.27 1.27)) (justify left bottom))
   )
-  (global_label "SC-" (shape input) (at 44.45 58.42 0) (fields_autoplaced)
-    (effects (font (size 1.27 1.27)) (justify left))
-    (property "Intersheet References" "${INTERSHEET_REFS}" (id 0) (at 50.915 58.3406 0)
-      (effects (font (size 1.27 1.27)) (justify left) hide)
-    )
-  )
   (global_label "SC+" (shape input) (at 129.54 59.69 0) (fields_autoplaced)
     (effects (font (size 1.27 1.27)) (justify left))
@@
     )
   )
-  (global_label "SC-" (shape input) (at 129.54 80.01 0) (fields_autoplaced)
-    (effects (font (size 1.27 1.27)) (justify left))
-    (property "Intersheet References" "${INTERSHEET_REFS}" (id 0) (at 136.005 79.9306 0)
-      (effects (font (size 1.27 1.27)) (justify left) hide)
-    )
-  )
   (global_label "SC+" (shape input) (at 129.54 73.66 0) (fields_autoplaced)
     (effects (font (size 1.27 1.27)) (justify left))
@@
     )
   )
-  (global_label "SC-" (shape input) (at 129.54 62.23 0) (fields_autoplaced)
-    (effects (font (size 1.27 1.27)) (justify left))
-    (property "Intersheet References" "${INTERSHEET_REFS}" (id 0) (at 136.005 62.1506 0)
-      (effects (font (size 1.27 1.27)) (justify left) hide)
-    )
-  )
   (symbol (lib_id "Mechanical:MountingHole") (at 62.23 97.79 0) (unit 1)
     (in_bom yes) (on_board yes) (fields_autoplaced)
@@
     )
   )
+  (symbol (lib_id "power:GND") (at 121.92 80.01 0) (unit 1)
+    (in_bom yes) (on_board yes)
+    (property "Reference" "#PWR?" (id 0) (at 121.92 86.36 0)
+      (effects (font (size 1.27 1.27)) hide)
+    )
+    (property "Value" "GND" (id 1) (at 127 81.28 0))
+    (property "Footprint" "" (id 2) (at 121.92 80.01 0)
+      (effects (font (size 1.27 1.27)) hide)
+    )
+    (property "Datasheet" "" (id 3) (at 121.92 80.01 0)
+      (effects (font (size 1.27 1.27)) hide)
+    )
+    (pin "1")
+  )
   (symbol (lib_id "Mechanical:MountingHole") (at 40.64 97.79 0) (unit 1)
     (in_bom yes) (on_board yes) (fields_autoplaced)
@@
     )
   )
+  (symbol (lib_id "power:GND") (at 121.92 62.23 0) (unit 1)
+    (in_bom yes) (on_board yes)
+    (property "Reference" "#PWR?" (id 0) (at 121.92 68.58 0)
+      (effects (font (size 1.27 1.27)) hide)
+    )
+    (property "Value" "GND" (id 1) (at 127 63.5 0))
+    (property "Footprint" "" (id 2) (at 121.92 62.23 0)
+      (effects (font (size 1.27 1.27)) hide)
+    )
+    (property "Datasheet" "" (id 3) (at 121.92 62.23 0)
+      (effects (font (size 1.27 1.27)) hide)
+    )
+    (pin "1")
+  )
   (symbol (lib_id "Mechanical:MountingHole") (at 62.23 115.57 0) (unit 1)
     (in_bom yes) (on_board yes) (fields_autoplaced)
@@
     )
     (property "DNP" "DNP" (id 4) (at 44.45 58.42 90)
+      (effects (font (size 1.27 1.27)) hide)
+    )
+    (pin "1")
+  )
+  (symbol (lib_id "power:GND") (at 45.72 58.42 0) (unit 1)
+    (in_bom yes) (on_board yes)
+    (property "Reference" "#PWR?" (id 0) (at 45.72 64.77 0)
+      (effects (font (size 1.27 1.27)) hide)
+    )
+    (property "Value" "GND" (id 1) (at 50.8 59.69 0))
+    (property "Footprint" "" (id 2) (at 45.72 58.42 0)
+      (effects (font (size 1.27 1.27)) hide)
+    )
+    (property "Datasheet" "" (id 3) (at 45.72 58.42 0)
       (effects (font (size 1.27 1.27)) hide)
     )
@@
   )
   (symbol_instances
+    (path "/0f7d02c9-1bea-47bd-8909-59bb88f849f3"
+      (reference "#PWR?") (unit 1) (value "GND") (footprint "")
+    )
+    (path "/371e6342-ad1d-4543-9f9c-c04defffdf9d"
+      (reference "#PWR?") (unit 1) (value "GND") (footprint "")
+    )
+    (path "/b1a648ae-90d0-44ef-954e-506f6bf8b472"
+      (reference "#PWR?") (unit 1) (value "GND") (footprint "")
+    )
     (path "/bb8f08ee-7552-4fc5-ba73-0c323731d189"
       (reference "H1") (unit 1) (value "MountingHole") (footprint "MountingHole:MountingHole_3.2mm_M3_DIN965_Pad")
