File: solar-cells/solar-cell-non-usb-side/solar-cell-pcbs-usb.kicad_pcb (KiCad board)
At the start: 2 copper layers, 80 x 103.5 mm, 13 parts, among them J1 Solar Cell

Commit message: added more annotations
Routing:
- net GND: track 0.00 -> 0.84 mm
Changed lines of the file:
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@@
+  )
+  (dimension (type aligned) (layer "Dwgs.User")
+    (pts (xy 82.6 66.55) (xy 82.6 70.05))
+    (height 22.1)
+    (gr_text "3.5000 mm" (at 58.7 68.3 90) (layer "Dwgs.User")
+      (effects (font (size 1.5 1.5) (thickness 0.3)))
+    )
+    (format (units 3) (units_format 1) (precision 4))
+    (style (thickness 0.2) (arrow_length 1.27) (text_position_mode 0) (extension_height 0.58642) (extension_offset 0.5) keep_text_aligned)
   )
   (dimension (type aligned) (layer "Dwgs.User")
@@
     (height -6.5)
     (gr_text "5.0000 mm" (at 67.7 50.75 90) (layer "Dwgs.User")
+      (effects (font (size 1.5 1.5) (thickness 0.3)))
+    )
+    (format (units 3) (units_format 1) (precision 4))
+    (style (thickness 0.2) (arrow_length 1.27) (text_position_mode 0) (extension_height 0.58642) (extension_offset 0.5) keep_text_aligned)
+  )
+  (dimension (type aligned) (layer "Dwgs.User")
+    (pts (xy 82.6 110.95) (xy 82.6 114.45))
+    (height 21.85)
+    (gr_text "3.5000 mm" (at 58.95 112.7 90) (layer "Dwgs.User")
       (effects (font (size 1.5 1.5) (thickness 0.3)))
     )
@@
   (via (at 97.275 121.25) (size 0.8) (drill 0.4) (layers "F.Cu" "B.Cu") (free) (net 1))
   (via (at 99.775 117.075) (size 0.8) (drill 0.4) (layers "F.Cu" "B.Cu") (free) (net 1))
+  (segment (start 82.5 68) (end 82.5 68.2) (width 0.25) (layer "B.Cu") (net 1))
+  (segment (start 82.5 68) (end 82.25 68) (width 1.27) (layer "B.Cu") (net 1))
+  (segment (start 82.5 68) (end 82.5 68.25) (width 1.27) (layer "B.Cu") (net 1))
+  (segment (start 82.5 68.2) (end 82.6 68.3) (width 0.25) (layer "B.Cu") (net 1))
   (segment (start 91.199999 112.7) (end 82.6 112.7) (width 1.27) (layer "B.Cu") (net 2))
   (segment (start 94.999999 116.5) (end 91.199999 112.7) (width 1.27) (layer "B.Cu") (net 2))

Commit message: changes to non usb side
Routing:
- net GND: track 0.84 -> 77.1 mm, vias 12 -> 0
- removed copper zone on B.Cu, net GND
Changed lines of the file:
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@@
     (style (thickness 0.15) (arrow_length 1.27) (text_position_mode 0) (extension_height 0.58642) (extension_offset 0.5) keep_text_aligned)
   )
-  (via (at 85.325 71.75) (size 0.8) (drill 0.4) (layers "F.Cu" "B.Cu") (free) (net 1))
-  (via (at 97.325 119.6) (size 0.8) (drill 0.4) (layers "F.Cu" "B.Cu") (free) (net 1))
-  (via (at 86.125 64.725) (size 0.8) (drill 0.4) (layers "F.Cu" "B.Cu") (free) (net 1))
-  (via (at 101.225 118.825) (size 0.8) (drill 0.4) (layers "F.Cu" "B.Cu") (free) (net 1))
-  (via (at 99.85 115.325) (size 0.8) (drill 0.4) (layers "F.Cu" "B.Cu") (free) (net 1))
-  (via (at 99.25 118.825) (size 0.8) (drill 0.4) (layers "F.Cu" "B.Cu") (free) (net 1))
-  (via (at 82.7 72.425) (size 0.8) (drill 0.4) (layers "F.Cu" "B.Cu") (free) (net 1))
-  (via (at 82.95 63.925) (size 0.8) (drill 0.4) (layers "F.Cu" "B.Cu") (free) (net 1))
-  (via (at 87.5 70.15) (size 0.8) (drill 0.4) (layers "F.Cu" "B.Cu") (free) (net 1))
-  (via (at 87.65 67.25) (size 0.8) (drill 0.4) (layers "F.Cu" "B.Cu") (free) (net 1))
-  (via (at 97.275 121.25) (size 0.8) (drill 0.4) (layers "F.Cu" "B.Cu") (free) (net 1))
-  (via (at 99.775 117.075) (size 0.8) (drill 0.4) (layers "F.Cu" "B.Cu") (free) (net 1))
-  (segment (start 82.5 68) (end 82.5 68.2) (width 0.25) (layer "B.Cu") (net 1))
-  (segment (start 82.5 68) (end 82.25 68) (width 1.27) (layer "B.Cu") (net 1))
-  (segment (start 82.5 68) (end 82.5 68.25) (width 1.27) (layer "B.Cu") (net 1))
-  (segment (start 82.5 68.2) (end 82.6 68.3) (width 0.25) (layer "B.Cu") (net 1))
+  (segment (start 82.6 101.005001) (end 82.6 68.3) (width 1.27) (layer "B.Cu") (net 1))
+  (segment (start 76 48.15) (end 82.6 54.75) (width 1.27) (layer "B.Cu") (net 1))
+  (segment (start 82.525 101.080001) (end 97 115.555001) (width 1.27) (layer "B.Cu") (net 1))
+  (segment (start 97 115.555001) (end 97 116.5) (width 1.27) (layer "B.Cu") (net 1))
+  (segment (start 82.525 101.080001) (end 82.6 101.005001) (width 1.27) (layer "B.Cu") (net 1))
+  (segment (start 82.6 54.75) (end 82.6 68.3) (width 1.27) (layer "B.Cu") (net 1))
   (segment (start 91.199999 112.7) (end 82.6 112.7) (width 1.27) (layer "B.Cu") (net 2))
   (segment (start 94.999999 116.5) (end 91.199999 112.7) (width 1.27) (layer "B.Cu") (net 2))
   (segment (start 75.95 106.05) (end 75.95 53.25) (width 1.27) (layer "B.Cu") (net 2))
   (segment (start 82.6 112.7) (end 75.95 106.05) (width 1.27) (layer "B.Cu") (net 2))
-  (zone (net 1) (net_name "GND") (layer "B.Cu") (hatch edge 0.508)
-    (connect_pads (clearance 0.508))
-    (min_thickness 0.254) (filled_areas_thickness no)
-    (fill yes (thermal_gap 0.508) (thermal_bridge_width 0.508))
-    (polygon
-      (pts
-        (xy 152.9 37.775)
-        (xy 153.075 143.475)
-        (xy 70.975 143.5)
-        (xy 70.925 37.625)
-        (xy 70.925 37.6)
-      )
-    )
-  )
 )
