File: solar-cells/new-solar-cell-burn-wire/new-solar-cell-burn-wire.kicad_pcb (KiCad board)
At the start: 2 copper layers, 80 x 103.5 mm, 29 parts, among them J1 Solar Cell, J2 Burn Wire

Commit message: modify pcb
Routing:
- net Net-(D1-Pad2): track 82.2 -> 88.0 mm
Changed lines of the file:
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@@
       (effects (font (size 1 1) (thickness 0.15)))
     )
-    (fp_text user "+" (at 8.89 -5.58) (layer "F.SilkS")
+    (fp_text user "+" (at 8.89 -5.58) (layer "B.SilkS")
       (effects (font (size 3 3) (thickness 0.3)))
     )
-    (fp_text user "-" (at 8.89 4.58 90) (layer "F.SilkS")
+    (fp_text user "-" (at 8.89 4.58 90) (layer "B.SilkS")
       (effects (font (size 3 3) (thickness 0.3)))
     )
@@
       (effects (font (size 1 1) (thickness 0.15)))
     )
-    (fp_text user "+" (at 8.89 -5.58) (layer "F.SilkS")
+    (fp_text user "+" (at 8.89 -5.58) (layer "B.SilkS")
       (effects (font (size 3 3) (thickness 0.3)))
     )
-    (fp_text user "-" (at 8.89 4.58 90) (layer "F.SilkS")
+    (fp_text user "-" (at 8.89 4.58 90) (layer "B.SilkS")
       (effects (font (size 3 3) (thickness 0.3)))
     )
@@
       (effects (font (size 1 1) (thickness 0.15)))
     )
-    (fp_text user "-" (at 8.89 4.58 90) (layer "F.SilkS")
+    (fp_text user "-" (at 8.89 4.58 90) (layer "B.SilkS")
       (effects (font (size 3 3) (thickness 0.3)))
     )
-    (fp_text user "+" (at 8.89 -5.58) (layer "F.SilkS")
+    (fp_text user "+" (at 8.89 -5.58) (layer "B.SilkS")
       (effects (font (size 3 3) (thickness 0.3)))
     )
@@
     (property "Sheetname" "")
     (attr through_hole)
-    (fp_text reference "J1" (at -0.95 -3.65) (layer "B.SilkS")
+    (fp_text reference "J1" (at -0.95 -3.65) (layer "B.Fab")
       (effects (font (size 1 1) (thickness 0.15)) (justify mirror))
     )
-    (fp_text value "Solar Cell" (at -1.1035 9.824999) (layer "B.SilkS")
+    (fp_text value "Solar Cell" (at -1.05 -3.85) (layer "B.SilkS")
       (effects (font (size 1 1) (thickness 0.15)) (justify mirror))
     )
@@
     (property "Sheetname" "")
     (attr through_hole)
-    (fp_text reference "J2" (at -1.05 -3.65) (layer "B.SilkS")
+    (fp_text reference "J2" (at -1.05 -3.65) (layer "B.Fab")
       (effects (font (size 1 1) (thickness 0.15)) (justify mirror))
     )
-    (fp_text value "Burn Wire" (at -1.043495 9.824999) (layer "B.SilkS")
+    (fp_text value "Burn Wire" (at -1.043495 -3.85) (layer "B.SilkS")
       (effects (font (size 1 1) (thickness 0.15)) (justify mirror))
     )
@@
   (gr_line (start 80.6 142.25) (end 80.6 135.9) (layer "Edge.Cuts") (width 0.1))
   (gr_line (start 137.25 46.75) (end 141.95 46.75) (layer "Edge.Cuts") (width 0.1))
+  (gr_text "+" (at 142.4 84.6) (layer "B.SilkS")
+    (effects (font (size 3 3) (thickness 0.3)) (justify mirror))
+  )
+  (gr_text "-" (at 107 117.6 -90) (layer "B.SilkS")
+    (effects (font (size 3 3) (thickness 0.3)) (justify mirror))
+  )
+  (gr_text "-" (at 142.8 94.8 -90) (layer "B.SilkS")
+    (effects (font (size 3 3) (thickness 0.3)) (justify mirror))
+  )
   (gr_text "+" (at 102.35 120.575) (layer "B.SilkS")
     (effects (font (size 1.5 1.5) (thickness 0.3)) (justify mirror))
   )
+  (gr_text "+" (at 106.6 84.64) (layer "B.SilkS")
+    (effects (font (size 3 3) (thickness 0.3)) (justify mirror))
+  )
   (gr_text "-" (at 87.75 120.775 -180) (layer "B.SilkS")
     (effects (font (size 1.5 1.5) (thickness 0.3)) (justify mirror))
@@
     (effects (font (size 1.5 1.5) (thickness 0.3)) (justify mirror))
   )
+  (gr_text "-" (at 107 94.8 -90) (layer "B.SilkS")
+    (effects (font (size 3 3) (thickness 0.3)) (justify mirror))
+  )
+  (gr_text "+" (at 106.6 107.44) (layer "B.SilkS")
+    (effects (font (size 3 3) (thickness 0.3)) (justify mirror))
+  )
   (gr_text "MOMOBOT" (at 112.2 140.6) (layer "F.SilkS")
     (effects (font (size 1 1) (thickness 0.15)))
+  )
+  (gr_text "+" (at 142.4 61.8) (layer "F.SilkS")
+    (effects (font (size 3 3) (thickness 0.3)))
+  )
+  (gr_text "+" (at 142.4 107.44) (layer "F.SilkS")
+    (effects (font (size 3 3) (thickness 0.3)))
+  )
+  (gr_text "-" (at 142.4 71.96 90) (layer "F.SilkS")
+    (effects (font (size 3 3) (thickness 0.3)))
+  )
+  (gr_text "-" (at 142.4 117.6 90) (layer "F.SilkS")
+    (effects (font (size 3 3) (thickness 0.3)))
+  )
+  (gr_text "+" (at 106.6 61.8) (layer "F.SilkS")
+    (effects (font (size 3 3) (thickness 0.3)))
+  )
+  (gr_text "-" (at 106.6 72 90) (layer "F.SilkS")
+    (effects (font (size 3 3) (thickness 0.3)))
   )
   (dimension (type aligned) (layer "Dwgs.User")
@@
   (segment (start 76 110) (end 76 105.5) (width 0.5) (layer "F.Cu") (net 3))
   (segment (start 76 110) (end 78 108) (width 0.5) (layer "F.Cu") (net 3))
+  (segment (start 115.5 98.5) (end 116.7 99.7) (width 0.5) (layer "F.Cu") (net 4))
+  (segment (start 116.7 97.9) (end 116.7 97.3) (width 0.5) (layer "F.Cu") (net 4))
+  (segment (start 116.7 98.5) (end 116.7 97.9) (width 0.5) (layer "F.Cu") (net 4))
+  (segment (start 115.3 98.5) (end 115.6 98.5) (width 0.5) (layer "F.Cu") (net 4))
+  (segment (start 116.1 98.5) (end 116.7 99.1) (width 0.5) (layer "F.Cu") (net 4))
   (segment (start 77.5 98.5) (end 113.9 98.5) (width 0.5) (layer "F.Cu") (net 4))
-  (segment (start 116.7 101.1) (end 114.1 98.5) (width 0.5) (layer "F.Cu") (net 4))
-  (segment (start 116.7 111) (end 116.7 101.1) (width 0.5) (layer "F.Cu") (net 4))
-  (segment (start 114.1 98.5) (end 113.9 98.5) (width 0.5) (layer "F.Cu") (net 4))
-  (segment (start 113.9 98.5) (end 116.7 95.7) (width 0.5) (layer "F.Cu") (net 4))
+  (segment (start 115.3 98.5) (end 115.5 98.5) (width 0.5) (layer "F.Cu") (net 4))
+  (segment (start 113.9 98.5) (end 115.3 98.5) (width 0.5) (layer "F.Cu") (net 4))
+  (segment (start 116.7 99.1) (end 116.7 99.2) (width 0.5) (layer "F.Cu") (net 4))
   (segment (start 76 97) (end 77.5 98.5) (width 0.5) (layer "F.Cu") (net 4))
+  (segment (start 116.1 98.5) (end 116.7 98.5) (width 0.5) (layer "F.Cu") (net 4))
+  (segment (start 116.1 98.5) (end 116.7 97.9) (width 0.5) (layer "F.Cu") (net 4))
+  (segment (start 116.7 111) (end 116.7 99.7) (width 0.5) (layer "F.Cu") (net 4))
   (segment (start 76 97) (end 76 101.5) (width 0.5) (layer "F.Cu") (net 4))
+  (segment (start 110.7 117) (end 116.7 111) (width 0.5) (layer "F.Cu") (net 4))
+  (segment (start 115.6 98.5) (end 116.1 98.5) (width 0.5) (layer "F.Cu") (net 4))
+  (segment (start 116.7 99.7) (end 116.7 99.2) (width 0.5) (layer "F.Cu") (net 4))
+  (segment (start 116.7 97.3) (end 116.7 91.2) (width 0.5) (layer "F.Cu") (net 4))
   (segment (start 116.7 91.2) (end 110.7 85.2) (width 0.5) (layer "F.Cu") (net 4))
-  (segment (start 110.7 117) (end 116.7 111) (width 0.5) (layer "F.Cu") (net 4))
-  (segment (start 116.7 95.7) (end 116.7 91.2) (width 0.5) (layer "F.Cu") (net 4))
+  (segment (start 116.7 99.2) (end 116.7 98.5) (width 0.5) (layer "F.Cu") (net 4))
+  (segment (start 115.5 98.5) (end 116.7 97.3) (width 0.5) (layer "F.Cu") (net 4))
   (segment (start 76 88.5) (end 105 88.5) (width 0.5) (layer "F.Cu") (net 5))
   (segment (start 76 93) (end 76 88.5) (width 0.5) (layer "F.Cu") (net 5))
