File: antenna/antenna-solar-pcb/antenna-solar-pcb.kicad_pcb (KiCad board)
At the start: 2 copper layers, 97 x 97 mm, 21 parts, among them J1 SMA Connector Male, J2 Solar Cell, U1 HHM1589D1

Commit message: added screw holes for antennas in antenna-solar
Routing:
- net GND: vias 174 -> 183
Other:
- outline, holes or cut-outs redrawn
- board text added: "+"
- board text added: "-"
Changed lines of the file:
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@@
       (effects (font (size 1 1) (thickness 0.15)))
     )
-    (fp_text user "+" (at 8.89 -5.58 90) (layer "F.SilkS")
-      (effects (font (size 3 3) (thickness 0.3)))
+    (fp_text user "+" (at 8.89 -5.58 -270) (layer "B.SilkS")
+      (effects (font (size 3 3) (thickness 0.3)) (justify mirror))
     )
     (fp_text user "-" (at 8.89 4.58) (layer "F.SilkS")
@@
   (gr_line (start 165.5 59) (end 165.5 65.9) (layer "Edge.Cuts") (width 0.1))
   (gr_line (start 150.1 55.2) (end 150.1 52.5) (layer "Edge.Cuts") (width 0.1))
+  (gr_circle (center 118.5 86.7) (end 121.2 86.7) (layer "Edge.Cuts") (width 0.1) (fill none))
   (gr_arc (start 150.1 55.2) (mid 149.807107 55.907107) (end 149.1 56.2) (layer "Edge.Cuts") (width 0.1))
   (gr_line (start 86.9 141.8) (end 86.9 144.5) (layer "Edge.Cuts") (width 0.1))
@@
   (gr_arc (start 86.9 144.5) (mid 86.607107 145.207107) (end 85.9 145.5) (layer "Edge.Cuts") (width 0.1))
   (gr_line (start 78 50.5) (end 78 50) (layer "Edge.Cuts") (width 0.1))
+  (gr_circle (center 118.5 110.3) (end 121.2 110.3) (layer "Edge.Cuts") (width 0.1) (fill none))
   (gr_line (start 70 139) (end 70.5 139) (layer "Edge.Cuts") (width 0.1))
   (gr_arc (start 70.5 58) (mid 71.207107 58.292893) (end 71.5 59) (layer "Edge.Cuts") (width 0.1))
@@
   (gr_arc (start 75.2 66.9) (mid 75.907107 67.192893) (end 76.2 67.9) (layer "Edge.Cuts") (width 0.1))
   (gr_line (start 78 147) (end 78 146.5) (layer "Edge.Cuts") (width 0.1))
+  (gr_text "-" (at 142.2 130.5 -180) (layer "B.SilkS")
+    (effects (font (size 3 3) (thickness 0.3)) (justify mirror))
+  )
+  (gr_text "+" (at 85.5 65.4) (layer "B.SilkS")
+    (effects (font (size 3 3) (thickness 0.3)) (justify mirror))
+  )
+  (gr_text "-" (at 95.5 66.1 -180) (layer "B.SilkS")
+    (effects (font (size 3 3) (thickness 0.3)) (justify mirror))
+  )
+  (gr_text "-" (at 84.5 131.7 -180) (layer "B.SilkS")
+    (effects (font (size 3 3) (thickness 0.3)) (justify mirror))
+  )
+  (gr_text "+" (at 94.9 131.1) (layer "B.SilkS")
+    (effects (font (size 3 3) (thickness 0.3)) (justify mirror))
+  )
+  (gr_text "+" (at 141.9 65.4) (layer "B.SilkS")
+    (effects (font (size 3 3) (thickness 0.3)) (justify mirror))
+  )
+  (gr_text "-" (at 151.9 66 -180) (layer "B.SilkS")
+    (effects (font (size 3 3) (thickness 0.3)) (justify mirror))
+  )
+  (gr_text "+" (at 152.6 129.9) (layer "F.SilkS")
+    (effects (font (size 3 3) (thickness 0.3)))
+  )
   (gr_text "HHM1589D1" (at 131.95 106.6 180) (layer "B.Fab")
     (effects (font (size 1 1) (thickness 0.15)) (justify mirror))
@@
   (via (at 125.35 93.35) (size 0.8) (drill 0.4) (layers "F.Cu" "B.Cu") (free) (net 3))
   (via (at 133.3 95.05) (size 0.8) (drill 0.4) (layers "F.Cu" "B.Cu") (free) (net 3))
+  (via (at 102.4 115.7) (size 0.8) (drill 0.4) (layers "F.Cu" "B.Cu") (free) (net 3))
   (via (at 102.05 113.95) (size 0.8) (drill 0.4) (layers "F.Cu" "B.Cu") (free) (net 3))
   (via (at 101.7 104.3) (size 0.8) (drill 0.4) (layers "F.Cu" "B.Cu") (free) (net 3))
@@
   (via (at 108.4 104.05) (size 0.8) (drill 0.4) (layers "F.Cu" "B.Cu") (free) (net 3))
   (via (at 106.65 103.1) (size 0.8) (drill 0.4) (layers "F.Cu" "B.Cu") (free) (net 3))
+  (via (at 128.6 103.6) (size 0.8) (drill 0.4) (layers "F.Cu" "B.Cu") (free) (net 3))
   (via (at 114.7 103.45) (size 0.8) (drill 0.4) (layers "F.Cu" "B.Cu") (free) (net 3))
   (via (at 104.8 94.35) (size 0.8) (drill 0.4) (layers "F.Cu" "B.Cu") (free) (net 3))
@@
   (via (at 135.05 94.2) (size 0.8) (drill 0.4) (layers "F.Cu" "B.Cu") (free) (net 3))
   (via (at 118.5 95.75) (size 0.8) (drill 0.4) (layers "F.Cu" "B.Cu") (free) (net 3))
+  (via (at 133.1 80.4) (size 0.8) (drill 0.4) (layers "F.Cu" "B.Cu") (free) (net 3))
   (via (at 121.1 81.45) (size 0.8) (drill 0.4) (layers "F.Cu" "B.Cu") (free) (net 3))
   (via (at 135.25 109) (size 0.8) (drill 0.4) (layers "F.Cu" "B.Cu") (free) (net 3))
@@
   (via (at 108.25 81.45) (size 0.8) (drill 0.4) (layers "F.Cu" "B.Cu") (free) (net 3))
   (via (at 136.95 100.85) (size 0.8) (drill 0.4) (layers "F.Cu" "B.Cu") (free) (net 3))
+  (via (at 104.1 116.6) (size 0.8) (drill 0.4) (layers "F.Cu" "B.Cu") (free) (net 3))
   (via (at 103.3 103.35) (size 0.8) (drill 0.4) (layers "F.Cu" "B.Cu") (free) (net 3))
   (via (at 113.45 94.8) (size 0.8) (drill 0.4) (layers "F.Cu" "B.Cu") (free) (net 3))
   (via (at 121.35 104.8) (size 0.8) (drill 0.4) (layers "F.Cu" "B.Cu") (free) (net 3))
   (via (at 111.65 101.3) (size 0.8) (drill 0.4) (layers "F.Cu" "B.Cu") (free) (net 3))
+  (via (at 128.6 93.4) (size 0.8) (drill 0.4) (layers "F.Cu" "B.Cu") (free) (net 3))
   (via (at 135.05 96.3) (size 0.8) (drill 0.4) (layers "F.Cu" "B.Cu") (free) (net 3))
+  (via (at 133 116.4) (size 0.8) (drill 0.4) (layers "F.Cu" "B.Cu") (free) (net 3))
   (via (at 106.55 100.85) (size 0.8) (drill 0.4) (layers "F.Cu" "B.Cu") (free) (net 3))
   (via (at 111.8 115.55) (size 0.8) (drill 0.4) (layers "F.Cu" "B.Cu") (free) (net 3))
@@
   (via (at 123 81.45) (size 0.8) (drill 0.4) (layers "F.Cu" "B.Cu") (free) (net 3))
   (via (at 113.65 81.45) (size 0.8) (drill 0.4) (layers "F.Cu" "B.Cu") (free) (net 3))
+  (via (at 104.1 79.5) (size 0.8) (drill 0.4) (layers "F.Cu" "B.Cu") (free) (net 3))
   (via (at 122.2 103.45) (size 0.8) (drill 0.4) (layers "F.Cu" "B.Cu") (free) (net 3))
   (via (at 105.05 104.3) (size 0.8) (drill 0.4) (layers "F.Cu" "B.Cu") (free) (net 3))
@@
   (via (at 106.4 93.15) (size 0.8) (drill 0.4) (layers "F.Cu" "B.Cu") (free) (net 3))
   (via (at 133.15 99.5) (size 0.8) (drill 0.4) (layers "F.Cu" "B.Cu") (free) (net 3))
+  (via (at 134.5 81.6) (size 0.8) (drill 0.4) (layers "F.Cu" "B.Cu") (free) (net 3))
   (via (at 103.15 92.85) (size 0.8) (drill 0.4) (layers "F.Cu" "B.Cu") (free) (net 3))
   (via (at 133 85.1) (size 0.8) (drill 0.4) (layers "F.Cu" "B.Cu") (free) (net 3))
@@
   (via (at 125.3 81.45) (size 0.8) (drill 0.4) (layers "F.Cu" "B.Cu") (free) (net 3))
   (via (at 122.2 93.55) (size 0.8) (drill 0.4) (layers "F.Cu" "B.Cu") (free) (net 3))
+  (via (at 135.2 115.7) (size 0.8) (drill 0.4) (layers "F.Cu" "B.Cu") (free) (net 3))
   (via (at 110.2 104.9) (size 0.8) (drill 0.4) (layers "F.Cu" "B.Cu") (free) (net 3))
   (via (at 123.05 115.55) (size 0.8) (drill 0.4) (layers "F.Cu" "B.Cu") (free) (net 3))
