File: solar-panels/Rip_my_life_pain_and_suffer_that_are_updated_board._Woe_is_my_name_struggle_is_my_life./new-solar-cell-usb-side/solar-cell-pcbs-usb.kicad_pcb (KiCad board)
At the start: 2 copper layers, 80 x 103.5 mm, 16 parts, among them J1 Solar Cell

Commit message: few touches and measurements to working solar panel usb side
Parts:
- removed H2, H3, H6: MountingHole_Pad, MountingHole:MountingHole_3.2mm_M3_DIN965_Pad
Changed lines of the file:
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@@
   (paper "A4")
   (title_block
-    (title "Solar Cell PCB (USB side)")
-    (date "2023-01-03")
-    (rev "3")
+    (title "Solar Panel (USB side)")
+    (date "2023-02-06")
+    (rev "4")
   )
   (layers
@@
       (net 7 "Net-(SC5-Pad2)") (pinfunction "-") (pintype "passive"))
   )
-  (footprint "MountingHole:MountingHole_3.2mm_M3_DIN965_Pad" (layer "F.Cu")
-    (at 125.85 42.75)
-    (descr "Mounting Hole 3.2mm, M3, DIN965")
-    (tags "mounting hole 3.2mm m3 din965")
-    (property "Sheetfile" "solar-cell-pcbs-usb.kicad_sch")
-    (property "Sheetname" "")
-    (attr exclude_from_pos_files)
-    (fp_text reference "H3" (at -5.95 -1.95) (layer "F.Fab")
-      (effects (font (size 1 1) (thickness 0.15)))
-    )
-    (fp_text value "MountingHole_Pad" (at 0 3.8) (layer "F.Fab")
-      (effects (font (size 1 1) (thickness 0.15)))
-    )
-    (fp_text user "${REFERENCE}" (at 0 0) (layer "F.Fab")
-      (effects (font (size 1 1) (thickness 0.15)))
-    )
-    (fp_circle (center 0 0) (end 2.8 0) (layer "Cmts.User") (width 0.15) (fill none))
-    (fp_circle (center 0 0) (end 3.05 0) (layer "F.CrtYd") (width 0.05) (fill none))
-    (pad "1" thru_hole circle (at 0 0) (size 5.6 5.6) (drill 3.2) (layers *.Cu *.Mask)
-      (net 1 "GND") (pinfunction "1") (pintype "input"))
-  )
   (footprint "ISP:SM101K07TF" (layer "F.Cu")
     (at 140.1 80.5 90)
@@
     (attr exclude_from_pos_files)
     (fp_text reference "H4" (at -4.5 -2.05) (layer "F.Fab")
-      (effects (font (size 1 1) (thickness 0.15)))
-    )
-    (fp_text value "MountingHole_Pad" (at 0 3.8) (layer "F.Fab")
-      (effects (font (size 1 1) (thickness 0.15)))
-    )
-    (fp_text user "${REFERENCE}" (at 0 0) (layer "F.Fab")
-      (effects (font (size 1 1) (thickness 0.15)))
-    )
-    (fp_circle (center 0 0) (end 2.8 0) (layer "Cmts.User") (width 0.15) (fill none))
-    (fp_circle (center 0 0) (end 3.05 0) (layer "F.CrtYd") (width 0.05) (fill none))
-    (pad "1" thru_hole circle (at 0 0) (size 5.6 5.6) (drill 3.2) (layers *.Cu *.Mask)
-      (net 1 "GND") (pinfunction "1") (pintype "input"))
-  )
-  (footprint "MountingHole:MountingHole_3.2mm_M3_DIN965_Pad" (layer "F.Cu")
-    (at 98.35 42.75)
-    (descr "Mounting Hole 3.2mm, M3, DIN965")
-    (tags "mounting hole 3.2mm m3 din965")
-    (property "Sheetfile" "solar-cell-pcbs-usb.kicad_sch")
-    (property "Sheetname" "")
-    (attr exclude_from_pos_files)
-    (fp_text reference "H2" (at -4.65 -2.2) (layer "F.Fab")
-      (effects (font (size 1 1) (thickness 0.15)))
-    )
-    (fp_text value "MountingHole_Pad" (at 0.15 3.95) (layer "F.Fab")
-      (effects (font (size 1 1) (thickness 0.15)))
-    )
-    (fp_text user "${REFERENCE}" (at 0 0) (layer "F.Fab")
-      (effects (font (size 1 1) (thickness 0.15)))
-    )
-    (fp_circle (center 0 0) (end 2.8 0) (layer "Cmts.User") (width 0.15) (fill none))
-    (fp_circle (center 0 0) (end 3.05 0) (layer "F.CrtYd") (width 0.05) (fill none))
-    (pad "1" thru_hole circle (at 0 0) (size 5.6 5.6) (drill 3.2) (layers *.Cu *.Mask)
-      (net 1 "GND") (pinfunction "1") (pintype "input"))
-  )
-  (footprint "MountingHole:MountingHole_3.2mm_M3_DIN965_Pad" (layer "F.Cu")
-    (at 98.35 138.25)
-    (descr "Mounting Hole 3.2mm, M3, DIN965")
-    (tags "mounting hole 3.2mm m3 din965")
-    (property "Sheetfile" "solar-cell-pcbs-usb.kicad_sch")
-    (property "Sheetname" "")
-    (attr exclude_from_pos_files)
-    (fp_text reference "H6" (at 0 -3.8) (layer "F.Fab")
       (effects (font (size 1 1) (thickness 0.15)))
     )
@@
   )
   (dimension (type aligned) (layer "Dwgs.User")
-    (pts (xy 98.35 138.25) (xy 125.85 138.25))
-    (height 23.25)
-    (gr_text "27.5000 mm" (at 112.1 160.35) (layer "Dwgs.User")
+    (pts (xy 84.6 138.25) (xy 139.6 138.25))
+    (height 13.449999)
+    (gr_text "55.0000 mm" (at 112.1 150.549999) (layer "Dwgs.User")
       (effects (font (size 1 1) (thickness 0.15)))
     )
     (format (units 3) (units_format 1) (precision 4))
     (style (thickness 0.15) (arrow_length 1.27) (text_position_mode 0) (extension_height 0.58642) (extension_offset 0.5) keep_text_aligned)
-  )
-  (dimension (type aligned) (layer "Dwgs.User")
-    (pts (xy 125.85 42.75) (xy 139.6 42.75))
-    (height -14.65)
-    (gr_text "13.7500 mm" (at 132.725 26.95) (layer "Dwgs.User")
-      (effects (font (size 1 1) (thickness 0.15)))
-    )
-    (format (units 3) (units_format 1) (precision 4))
-    (style (thickness 0.15) (arrow_length 1.27) (text_position_mode 0) (extension_height 0.58642) (extension_offset 0.5) keep_text_aligned)
-  )
-  (dimension (type aligned) (layer "Dwgs.User")
-    (pts (xy 125.85 138.25) (xy 139.6 138.25))
-    (height 16.85)
-    (gr_text "13.7500 mm" (at 132.725 153.95) (layer "Dwgs.User")
-      (effects (font (size 1 1) (thickness 0.15)))
-    )
-    (format (units 3) (units_format 1) (precision 4))
-    (style (thickness 0.15) (arrow_length 1.27) (text_position_mode 0) (extension_height 0.58642) (extension_offset 0.5) keep_text_aligned)
-  )
-  (dimension (type aligned) (layer "Dwgs.User")
-    (pts (xy 98.35 42.75) (xy 125.85 42.75))
-    (height -10.15)
-    (gr_text "27.5000 mm" (at 112.1 31.45) (layer "Dwgs.User")
-      (effects (font (size 1 1) (thickness 0.15)))
-    )
-    (format (units 3) (units_format 1) (precision 4))
-    (style (thickness 0.15) (arrow_length 1.27) (text_position_mode 0) (extension_height 0.58642) (extension_offset 0.5) keep_text_aligned)
-  )
-  (dimension (type aligned) (layer "Dwgs.User")
-    (pts (xy 84.6 138.25) (xy 98.35 138.25))
-    (height 18.45)
-    (gr_text "13.7500 mm" (at 91.475 155.55) (layer "Dwgs.User")
-      (effects (font (size 1 1) (thickness 0.15)))
-    )
-    (format (units 3) (units_format 1) (precision 4))
-    (style (thickness 0.15) (arrow_length 1.27) (text_position_mode 0) (extension_height 0.58642) (extension_offset 0.5) keep_text_aligned)
-  )
-  (dimension (type aligned) (layer "Dwgs.User")
-    (pts (xy 82.6 66.55) (xy 82.6 70.05))
-    (height 22.1)
-    (gr_text "3.5000 mm" (at 58.7 68.3 90) (layer "Dwgs.User")
-      (effects (font (size 1.5 1.5) (thickness 0.3)))
-    )
-    (format (units 3) (units_format 1) (precision 4))
-    (style (thickness 0.2) (arrow_length 1.27) (text_position_mode 0) (extension_height 0.58642) (extension_offset 0.5) keep_text_aligned)
   )
   (dimension (type aligned) (layer "Dwgs.User")
@@
   )
   (dimension (type aligned) (layer "Dwgs.User")
-    (pts (xy 84.6 42.75) (xy 98.35 42.75))
-    (height -10.15)
-    (gr_text "13.7500 mm" (at 91.475 31.45) (layer "Dwgs.User")
-      (effects (font (size 1 1) (thickness 0.15)))
-    )
+    (pts (xy 84.6 42.75) (xy 139.6 42.75))
+    (height -15.45)
+    (gr_text "55.0000 mm" (at 112.1 26.15) (layer "Dwgs.User")
+      (effects (font (size 1 1) (thickness 0.15)))
+    )
