File: solar-panels/Rip_my_life_pain_and_suffer_that_are_updated_board._Woe_is_my_name_struggle_is_my_life./new-solar-cell-usb-side/solar-cell-pcbs-usb.kicad_sch (KiCad schematic)
At the start: 16 parts, among them J1 Solar Cell

Commit message: few touches and measurements to working solar panel usb side
Parts:
- removed H2, H3, H6: MountingHole_Pad, MountingHole:MountingHole_3.2mm_M3_DIN965_Pad, symbol Mechanical:MountingHole_Pad
Other:
- title: Solar Cell PCB - usb side -> Solar Panel (USB Side)
- moved on the sheet: H4, H5, H7, J1
