File: bottom-adapter/bottom-adapter.kicad_pcb (KiCad board)
At the start: 2 copper layers, 97 x 97 mm, 15 parts, among them J2 Burn Wire

Commit message: Fixed names
Other:
- board text added: "Alex Kelso|Dr.S. & Raji Yegnasubramanian|Ethan Philpott|Rachel & Bella Philpott Bob & Joy Philpott|Robby & Angie Philpott|Dee Biggs|Rolo|Pablo Lazo|Kavitha Rau Tony & Mary Kelso|Zhang Guangmei|Tian Yonghui|Wang Linsen|Yuxuan & Ping Wang Dara Wang|Jacob Tall|Anu & Mahesh Saptharishi|Danfeng Xu|Gopal Rau|Amy Rao Satish & Lakshmi Yegnasubramanian|Thomas Cuvillier|Dongfeng Xu|Alex Xu|Liliana Abreu So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"
- board text added: "The Richman Family|Dr.H. & Rekha Rao|Savita Raj & Santosh Shastri|Dan Ellis|Don Lemon Nikita Bier|James Wilson|Jerry Wu|Shadow, Ethan's Snail & Fish, & Jìnzhǎn|Gold, Rachel's Fish, & Kitty|Michael & Joanne Chiglinsky|Roger & Dorothy Truslow|Letcher & Geraldine Philpott Arianne Abreu|Michael Bretti|Mateo Graziosi|Momoe Nomoto|Geethe & Nallicheri Shivagiri Jian T. Yang|Jihan Shende|Emily Hsieh|Andr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"
- board text removed: "Alex Kelso|Dr.S. & Raji Yegnasubramanian|Ethan Philpott|Rachel & Bella Philpott Bob & Joy Philpott|Robby,Angie & Dee Philpott|Rolo|Pablo Lazo|Kavitha Rau Tony & Mary Kelso|Zhang Guangmei|Tian Yonghui|Wang Linsen|Yuxuan & Ping Wang Dara Wang|Jacob Tall|Anu & Mahesh Saptharishi|Danfeng Xu|Gopal Rau|Amy Rao Satish & Lakshmi Yegnasubramanian|Thomas Cuvillier|Dongfeng Xu|Alex Xu|Liliana Abreu Soundari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"
- board text removed: "The Richman Family|Dr.H. & Rekha Rao|Savita Raj & Santosh Shastri|Dan Ellis|Don Lemon Nikita Bier|James Wilson|Jerry Wu|Shadow, Ethan's Snail & Fish, & Jìnzhǎn|Gold, Rachel's Fish, & Kitty|Michael Chiglinsky|Roger & Dorothy Truslow|Letcher & Geraldine Philpott Arianne Abreu|Michael Bretti|Mateo Graziosi|Momoe Nomoto|Geethe & Nallicheri Shivagiri Jian T. Yang|Jihan Shende|Emily Hsieh|Andrew Selep|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"
Changed lines of the file:
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@@
     (effects (font (size 1 1) (thickness 0.15)))
   )
-  (gr_text "\n\n\n\nAlex Kelso|Dr.S. & Raji Yegnasubramanian|Ethan Philpott|Rachel & Bella Philpott\nBob & Joy Philpott|Robby,Angie & Dee Philpott|Rolo|Pablo Lazo|Kavitha Rau\nTony & Mary Kelso|Zhang Guangmei|Tian Yonghui|Wang Linsen|Yuxuan & Ping Wang\nDara Wang|Jacob Tall|Anu & Mahesh Saptharishi|Danfeng Xu|Gopal Rau|Amy Rao\nSatish & Lakshmi Yegnasubramanian|Thomas Cuvillier|Dongfeng Xu|Alex Xu|Liliana Abreu\nSoundari & Murali Swaminathan|Mamtha Rau|Gopal & Sujatha Rau|Irvin Chadraa\nJuan Abreu|Prashanth Vasan|Naveen & Nayan Barriga|Bislim & Morena Ahmetaj\n\n" (at 116.84 66.04) (layer "F.SilkS")
+  (gr_text "\n\n\n\nAlex Kelso|Dr.S. & Raji Yegnasubramanian|Ethan Philpott|Rachel & Bella Philpott\nBob & Joy Philpott|Robby & Angie Philpott|Dee Biggs|Rolo|Pablo Lazo|Kavitha Rau\nTony & Mary Kelso|Zhang Guangmei|Tian Yonghui|Wang Linsen|Yuxuan & Ping Wang\nDara Wang|Jacob Tall|Anu & Mahesh Saptharishi|Danfeng Xu|Gopal Rau|Amy Rao\nSatish & Lakshmi Yegnasubramanian|Thomas Cuvillier|Dongfeng Xu|Alex Xu|Liliana Abreu\nSoundari & Murali Swaminathan|Mamtha Rau|Gopal & Sujatha Rau|Irvin Chadraa\nJuan Abreu|Prashanth Vasan|Naveen & Nayan Barriga|Bislim & Morena Ahmetaj\n\n" (at 116.84 66.04) (layer "F.SilkS")
     (effects (font (size 0.95 0.95) (thickness 0.1)))
   )
@@
     (effects (font (size 1 1) (thickness 0.15)))
   )
-  (gr_text "\n\nThe Richman Family|Dr.H. & Rekha Rao|Savita Raj & Santosh Shastri|Dan Ellis|Don Lemon\nNikita Bier|James Wilson|Jerry Wu|Shadow, Ethan's Snail & Fish, & Jìnzhǎn|Gold, Rachel's Fish,   \n& Kitty|Michael Chiglinsky|Roger & Dorothy Truslow|Letcher & Geraldine Philpott  \nArianne Abreu|Michael Bretti|Mateo Graziosi|Momoe Nomoto|Geethe & Nallicheri Shivagiri  \nJian T. Yang|Jihan Shende|Emily Hsieh|Andrew Selep|Sebastian Abreu|Santosh Rau  \nBob Jackson|Helen Xu|Alan Hentrich|Aiden Guo|Cheng Z. Liu|Jacqueline X. Yang  \n\n" (at 119.38 129.54) (layer "F.SilkS")
+  (gr_text "\n\nThe Richman Family|Dr.H. & Rekha Rao|Savita Raj & Santosh Shastri|Dan Ellis|Don Lemon\nNikita Bier|James Wilson|Jerry Wu|Shadow, Ethan's Snail & Fish, & Jìnzhǎn|Gold, Rachel's Fish,   \n& Kitty|Michael & Joanne Chiglinsky|Roger & Dorothy Truslow|Letcher & Geraldine Philpott  \nArianne Abreu|Michael Bretti|Mateo Graziosi|Momoe Nomoto|Geethe & Nallicheri Shivagiri  \nJian T. Yang|Jihan Shende|Emily Hsieh|Andrew Selep|Sebastian Abreu|Santosh Rau  \nBob Jackson|Helen Xu|Alan Hentrich|Aiden Guo|Cheng Z. Liu|Jacqueline X. Yang  \n\n" (at 119.38 129.54) (layer "F.SilkS")
     (effects (font (size 0.95 0.95) (thickness 0.10125)))
   )

Commit message: Added text for special thanks to
Other:
- board text added: "Oleg Shargorodskiy Professor Joseph Borowiec Michael Pham Flynn Dreilinger"
- board text added: "Special Thanks To:"
Changed lines of the file:
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@@
+    (effects (font (size 1 1) (thickness 0.15)) (justify mirror))
+  )
+  (gr_text "Special Thanks To:" (at 116.84 116.84) (layer "B.SilkS")
+    (effects (font (size 1.15 1.15) (thickness 0.23) bold) (justify mirror))
+  )
+  (gr_text "Oleg Shargorodskiy\nProfessor Joseph Borowiec \nMichael Pham \nFlynn Dreilinger" (at 116.84 121.92) (layer "B.SilkS")
     (effects (font (size 1 1) (thickness 0.15)) (justify mirror))
   )
