File: bottom-adapter/bottom-adapter.kicad_pcb (KiCad board)
At the start: 2 copper layers, 97 x 97 mm, 15 parts, among them J2 Burn Wire

Commit message: Added quotes
Other:
- board text added: "Quotes:"
- board text added: "{dblquote}God is love{dblquote} - Michael Chiglinsky {dblquote}Praise be to god{dblquote} - Ethan Philpott"
Changed lines of the file:
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@@
     (effects (font (size 1 1) (thickness 0.15)) (justify mirror))
   )
-  (gr_text "Special Thanks To:" (at 118.25 111.76) (layer "B.SilkS")
+  (gr_text "Special Thanks To:" (at 118.25 112) (layer "B.SilkS")
     (effects (font (size 1.15 1.15) (thickness 0.23) bold) (justify bottom mirror))
   )
+  (gr_text "Quotes:" (at 121.626071 132.08) (layer "B.SilkS")
+    (effects (font (size 1.15 1.15) (thickness 0.23) bold) (justify left bottom mirror))
+  )
+  (gr_text "{dblquote}God is love{dblquote} - Michael Chiglinsky\n{dblquote}Praise be to god{dblquote} - Ethan Philpott" (at 118.25 136.7) (layer "B.SilkS")
+    (effects (font (size 1 1) (thickness 0.15)) (justify bottom mirror))
+  )
   (gr_text "Oleg Shargorodskiy\nProfessor Joseph Borowiec \nMichael Pham \nFlynn Dreilinger" (at 118.25 119.38) (layer "B.SilkS")

Commit message: Fixed quote spacing kicad
Other:
- board text removed: "Oleg Shargorodskiy Professor Joseph Borowiec Michael Pham Flynn Dreilinger"
- board text removed: "{dblquote}God is love{dblquote} - Michael Chiglinsky {dblquote}Praise be to god{dblquote} - Ethan Philpott"
Changed lines of the file:
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@@
     (effects (font (size 1 1) (thickness 0.15)) (justify mirror))
+  )
+  (gr_text "Quotes:" (at 118.25 133.59) (layer "B.SilkS")
+    (effects (font (size 1.15 1.15) (thickness 0.23) bold) (justify bottom mirror))
   )
   (gr_text "GND\n" (at 112 101.6) (layer "B.SilkS")
@@
   (gr_text "Special Thanks To:" (at 118.25 112) (layer "B.SilkS")
     (effects (font (size 1.15 1.15) (thickness 0.23) bold) (justify bottom mirror))
-  )
-  (gr_text "Quotes:" (at 121.626071 132.08) (layer "B.SilkS")
-    (effects (font (size 1.15 1.15) (thickness 0.23) bold) (justify left bottom mirror))
-  )
-  (gr_text "{dblquote}God is love{dblquote} - Michael Chiglinsky\n{dblquote}Praise be to god{dblquote} - Ethan Philpott" (at 118.25 136.7) (layer "B.SilkS")
-    (effects (font (size 1 1) (thickness 0.15)) (justify bottom mirror))
-  )
-  (gr_text "Oleg Shargorodskiy\nProfessor Joseph Borowiec \nMichael Pham \nFlynn Dreilinger" (at 118.25 119.38) (layer "B.SilkS")
-    (effects (font (size 1 1) (thickness 0.15)) (justify bottom mirror))
   )
   (gr_text "\n\n\nRexforr|Bisser Paskalev|Srinidhi Ananth|Steffen Jauch\njcubic|Ryan W|Simran Hajarnavis|Xiqin Yang|Weiying Huang\nJulian Galaz|Kaylynn Yamanashi|Cassandra Riley|Ashok Sudarshanam\nLuca Richman|Alberto Lugo|Anthony Ucciferri| Michelle Hernandez\nEthan Taub|Jing Zhang|Charles Xie|Henry Cowherd|Chris Glenn\nSean|Madhura & Ranga Nadig|Geeta & Ramji Paranandi|Adam Kang\nGreg Panzer|Susan Post|Shobha Rao|Danny Breeze|Shawn Tolidano\nFiona Selep|Michael Ness|Pepito\n" (at 91.44 99.06 270) (layer "F.SilkS")
@@
     (effects (font (size 0.9 0.9) (thickness 0.10125)))
   )
+  (gr_text_box "Oleg Shargorodskiy\nProfessor Joseph Borowiec \nMichael Pham \nFlynn Dreilinger"
+    (start 101.74 113.03) (end 134.76 120.65) (layer "B.SilkS")
+      (effects (font (size 1 1) (thickness 0.15)) (justify top mirror))
+  )
+  (gr_text_box "{dblquote}God is love{dblquote} - Michael Chiglinsky\n{dblquote}Praise be to god{dblquote} - Ethan Philpott"
+    (start 101.74 134.62) (end 134.76 139.7) (layer "B.SilkS")
+      (effects (font (size 1 1) (thickness 0.15)) (justify top mirror))
+  )
   (dimension (type aligned) (layer "Dwgs.User")

Commit message: Removed quotes title
Other:
- board text removed: "Quotes:"
Changed lines of the file:
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@@
     (effects (font (size 1 1) (thickness 0.15)) (justify mirror))
-  )
-  (gr_text "Quotes:" (at 118.25 133.59) (layer "B.SilkS")
-    (effects (font (size 1.15 1.15) (thickness 0.23) bold) (justify bottom mirror))
   )
   (gr_text "GND\n" (at 112 101.6) (layer "B.SilkS")
@@
       (effects (font (size 1 1) (thickness 0.15)) (justify top mirror))
   )
-  (gr_text_box "{dblquote}God is love{dblquote} - Michael Chiglinsky\n{dblquote}Praise be to god{dblquote} - Ethan Philpott"
-    (start 101.74 134.62) (end 134.76 139.7) (layer "B.SilkS")
+  (gr_text_box "{dblquote}God is love{dblquote} - Michael Chiglinsky | {dblquote}Praise be to god{dblquote} - Ethan Philpott"
+    (start 82.69 137.16) (end 153.81 139.7) (layer "B.SilkS")
       (effects (font (size 1 1) (thickness 0.15)) (justify top mirror))
   )
