File: solar-panels/usb-side/solar-cell-pcbs-usb.kicad_pcb (KiCad board)
At the start: 2 copper layers, 80 x 103.5 mm, 13 parts, among them J1 Solar Cell

Commit message: local
Routing:
- net GND: track 0.00 -> 35.8 mm
- net (no net): vias 20 -> 18
